Commit message: add fixed model, make separate launch for joint_state_pub

File: project2_dhmanip/urdf/manip_fixed.urdf (robot description, URDF)
Before this commit: robot manipulator, 5 links, 4 joints
Joints:
- joint joint1: type revolute -> fixed
- joint joint2: type revolute -> fixed
- joint joint3: type revolute -> fixed
