Commit message: second robot version

File: project2_dhmanip/urdf/manip.urdf (robot description, URDF)
Before this commit: robot manipulator, 4 links, 3 joints
Links:
- added link link3; collision cylinder length=${d3} radius=${link_diam/2}; visual cylinder length=${d3} radius=${link_diam/2}
- link base_link: geometry collision cylinder length=${base_height} radius=${base_diam/2}; visual cylinder length=${base_height} radius=${base_diam/2}
- link link1: geometry collision cylinder length=${d1} radius=${link_diam/2}; visual cylinder length=${d1} radius=${link_diam/2}
- link link2: geometry collision cylinder length=${d2} radius=${link_diam/2}; visual cylinder length=${d2} radius=${link_diam/2}
Joints:
- added joint tool_joint: type fixed, parent link3, child tool, origin xyz=0 0 ${d3} rpy=1.5708 0 1.5708, axis 0 0 1, limit lower=-0.7 upper=3.8 effort=1000.0 velocity=0.5
- joint joint1: limit lower=0.0 upper=10 effort=1000.0 velocity=0.5 -> lower=-10 upper=10 effort=1000.0 velocity=0.5; origin xyz=0 0 ${d1} rpy=0 0 0 -> xyz=0 0 ${base_height} rpy=0 0 0
- joint joint2: limit lower=-0.7 upper=3.8 effort=1000.0 velocity=0.5 -> lower=-3.8 upper=3.8 effort=1000.0 velocity=0.5; origin xyz=0 0 ${d2} rpy=1.5708 0 1.5708 -> xyz=0 0 ${d1} rpy=1.5708 -1.5708 0
- joint joint3: child tool -> link3; limit lower=-0.7 upper=3.8 effort=1000.0 velocity=0.5 -> lower=-3.8 upper=3.8 effort=1000.0 velocity=0.5; origin xyz=0 0 ${d3} rpy=1.5708 0 1.5708 -> xyz=0 0 ${d2} rpy=1.5708 -1.5708 0

Commit message: add prismatic joints

File: project2_dhmanip/urdf/manip.urdf (robot description, URDF)
Before this commit: robot manipulator, 5 links, 4 joints
Joints:
- joint joint1: limit lower=-10 upper=10 effort=1000.0 velocity=0.5 -> lower=${-d1} upper=0 effort=1000.0 velocity=0.5; type revolute -> prismatic
- joint joint2: limit lower=-3.8 upper=3.8 effort=1000.0 velocity=0.5 -> lower=${-d2} upper=0 effort=1000.0 velocity=0.5; type revolute -> prismatic
- joint joint3: limit lower=-3.8 upper=3.8 effort=1000.0 velocity=0.5 -> lower=${-d3} upper=0 effort=1000.0 velocity=0.5; type revolute -> prismatic

Commit message: KOLEJNY

File: project2_dhmanip/urdf/manip.urdf (robot description, URDF)
Before this commit: robot manipulator, 5 links, 4 joints
Joints:
- joint joint2: origin xyz=0 0 ${d1} rpy=1.5708 -1.5708 0 -> xyz=0 0 ${d1} rpy=1.5708 -0.0 1.5708; type revolute -> prismatic
- joint joint3: origin xyz=0 0 ${d2} rpy=1.5708 -1.5708 0 -> xyz=0 0 ${d2} rpy=1.5708 -0.0 1.5708; type revolute -> prismatic
